Commit message: Made necessary changes for rviz simulation from xacro

File: p3dx_description/urdf/gz.xacro (robot description, xacro)
@@ -104,5 +104,5 @@
 	<gazebo reference="lms100">
 		<sensor type="gpu_lidar" name="gpu_lidar">
-			<topic>p3dx/scan</topic>
+			<topic>scan</topic>
 			<update_rate>50</update_rate>
 			<gz_frame_id>lms100</gz_frame_id>
@@ -118,5 +118,5 @@
 				</scan>
 				<range>
-					<min>0.10</min>
+					<min>0.20</min>
 					<max>30.0</max>
 					<resolution>0.01</resolution>

File: p3dx_description/urdf/p3dx.xacro (robot description, xacro)
@@ -6,8 +6,9 @@
 	<xacro:include filename="$(find p3dx_description)/urdf/p3dx_wheel.xacro" />
 	<!-- chassis -->
+	<link name="base" />
 	<link name="base_link">
 		<inertial>
 			<mass value="3.5" />
-			<origin xyz="-0.025 0 -0.223"/>
+			<!-- <origin xyz="-0.025 0 -0.223" /> -->
 			<origin xyz="-0.05 0 0" />
 			<inertia ixx="1" ixy="0" ixz="0" iyy="1" iyz="0" izz="1" />
@@ -16,5 +17,5 @@
 			<origin xyz="-0.045 0 0.148" rpy="0 0 0" />
 			<geometry name="pioneer_geom">
-				<mesh filename="$(find p3dx_description)/meshes/chassis.stl" />
+				<mesh filename="file://$(find p3dx_description)/meshes/chassis.stl" />
 			</geometry>
 			<material name="ChassisRed">
@@ -29,4 +30,9 @@
 		</collision>
 	</link>
+	<joint name="base_footprint_joint" type="fixed">
+		<origin xyz="0 0 0" rpy="0 0 0" />
+		<parent link="base" />
+		<child link="base_link" />
+	</joint>
 	<!-- top_plate -->
 	<link name="top_plate">
@@ -39,5 +45,5 @@
 			<origin xyz="0 0 0" rpy="0 0 0" />
 			<geometry name="top_geom">
-				<mesh filename="$(find p3dx_description)/meshes/top.stl" />
+				<mesh filename="file://$(find p3dx_description)/meshes/top.stl" />
 			</geometry>
 			<material name="TopBlack">
@@ -67,5 +73,5 @@
 			<origin xyz="0 0 0" rpy="0 0 0" />
 			<geometry name="pioneer_geom">
-				<mesh filename="$(find p3dx_description)/meshes/swivel.stl" />
+				<mesh filename="file://$(find p3dx_description)/meshes/swivel.stl" />
 			</geometry>
 			<material name="swivel">
@@ -100,5 +106,5 @@
 			<origin xyz="0 0 0" rpy="0 0 0" />
 			<geometry name="pioneer_geom">
-				<mesh filename="$(find p3dx_description)/meshes/center_hubcap.stl" />
+				<mesh filename="file://$(find p3dx_description)/meshes/center_hubcap.stl" />
 			</geometry>
 			<material name="swivel">
@@ -133,5 +139,5 @@
 			<origin xyz="0 0 0" rpy="0 0 0" />
 			<geometry name="pioneer_geom">
-				<mesh filename="$(find p3dx_description)/meshes/center_wheel.stl" />
+				<mesh filename="file://$(find p3dx_description)/meshes/center_wheel.stl" />
 			</geometry>
 			<material name="WheelBlack">
@@ -163,5 +169,5 @@
 			<origin rpy="0 0 0" xyz="0 0 0" />
 			<geometry name="pioneer_geom">
-				<mesh filename="$(find p3dx_description)/meshes/front_sonar.stl" />
+				<mesh filename="file://$(find p3dx_description)/meshes/front_sonar.stl" />
 			</geometry>
 			<material name="SonarYellow">
@@ -191,5 +197,5 @@
 			<origin xyz="0 0 0" rpy="0 0 0" />
 			<geometry>
-				<mesh filename="$(find p3dx_description)/meshes/lms100.dae" />
+				<mesh filename="file://$(find p3dx_description)/meshes/lms100.dae" />
 			</geometry>
 		</visual>

File: p3dx_description/urdf/p3dx_wheel.xacro (robot description, xacro)
@@ -15,5 +15,5 @@
 				<origin xyz="0 0 0" rpy="0 0 0" />
 				<geometry name="pioneer_geom">
-					<mesh filename="$(find p3dx_description)/meshes/${suffix}_hubcap.stl" />
+					<mesh filename="file://$(find p3dx_description)/meshes/${suffix}_hubcap.stl" />
 				</geometry>
 				<material name="HubcapYellow">
@@ -47,5 +47,5 @@
 				<origin xyz="0 0 0" rpy="0 0 0" />
 				<geometry name="pioneer_geom">
-					<mesh filename="$(find p3dx_description)/meshes/${suffix}_wheel.stl" />
+					<mesh filename="file://$(find p3dx_description)/meshes/${suffix}_wheel.stl" />
 				</geometry>
 				<material name="WheelBlack">
@@ -56,5 +56,5 @@
 				<origin xyz="0 0 0" rpy="${-3.1415927/2} 0 0" />
 				<geometry>
-					<!--<mesh filename="$(find p3dx_description)/meshes/${suffix}_wheel.stl"/> -->
+					<mesh filename="file://$(find p3dx_description)/meshes/${suffix}_wheel.stl"/>
 					<cylinder radius="0.09" length="0.01" />
 				</geometry>
@@ -84,5 +84,5 @@
 			<mu1>0.5</mu1>
 			<mu2>50.0</mu2>
-			<kp>100000000.0</kp>
+			<kp>1000.0</kp>
 			<kd>1.0</kd>
 		</gazebo>
