Commit message: Removed urdf, changed parent and child in wheels and hubcap joints

File: p3dx_description/urdf/p3dx_wheel.xacro (robot description, xacro)
@@ -5,4 +5,36 @@
 	<!-- right/left hubcap + wheel -->
 	<xacro:macro name="p3dx_wheel" params="suffix parent reflect">
+		<!-- hubcap -->
+		<link name="p3dx_${suffix}_hubcap">
+			<inertial>
+				<mass value="0.01" />
+				<origin xyz="0 0 0" />
+				<inertia ixx="0.012411765597" ixy="0" ixz="0" iyy="0.015218160428" iyz="0" izz="0.011763977943" />
+			</inertial>
+			<visual name="base_visual">
+				<origin xyz="0 0 0" rpy="0 0 0" />
+				<geometry name="pioneer_geom">
+					<mesh filename="$(find p3dx_description)/meshes/${suffix}_hubcap.stl" />
+				</geometry>
+				<material name="HubcapYellow">
+					<color rgba="1.0 0.811 0.151 1.0" />
+				</material>
+			</visual>
+			<collision>
+				<origin xyz="0 0 0" rpy="0 0 0" />
+				<geometry>
+					<box size="0.01 0.01 0.01" />
+				</geometry>
+			</collision>
+		</link>
+		<joint name="base_${suffix}_hubcap_joint" type="continuous">
+			<axis xyz="0 1 0" />
+			<anchor xyz="0 0 0" />
+			<limit effort="100" velocity="100" />
+			<joint_properties damping="0.0" friction="0.0" />
+			<origin xyz="0 ${reflect*0.158} 0.091" rpy="0 0 0" />
+			<parent link="base_link" />
+			<child link="p3dx_${suffix}_hubcap" />
+		</joint>
 		<!-- wheel -->
 		<link name="p3dx_${suffix}_wheel">
@@ -10,6 +42,5 @@
 				<mass value="0.5" />
 				<origin xyz="0 0 0" />
-				<inertia ixx="0.012411765597" ixy="0" ixz="0" iyy="0.015218160428"
-					iyz="0" izz="0.011763977943" />
+				<inertia ixx="0.012411765597" ixy="0" ixz="0" iyy="0.015218160428" iyz="0" izz="0.011763977943" />
 			</inertial>
 			<visual name="base_visual">
@@ -30,51 +61,18 @@
 			</collision>
 		</link>
-		<joint name="base_${suffix}_hubcap_joint" type="fixed">
+		<joint name="base_${suffix}_wheel_joint" type="fixed">
 			<origin xyz="0 0 0" rpy="0 0 0" />
-			<parent link="p3dx_${suffix}_wheel" />
-			<child link="p3dx_${suffix}_hubcap" />
-		</joint>
-		<!-- hubcap -->
-		<link name="p3dx_${suffix}_hubcap">
-			<inertial>
-				<mass value="0.01" />
-				<origin xyz="0 0 0" />
-				<inertia ixx="0.012411765597" ixy="0" ixz="0" iyy="0.015218160428"
-					iyz="0" izz="0.011763977943" />
-			</inertial>
-			<visual name="base_visual">
-				<origin xyz="0 0 0" rpy="0 0 0" />
-				<geometry name="pioneer_geom">
-					<mesh filename="$(find p3dx_description)/meshes/${suffix}_hubcap.stl" />
-				</geometry>
-				<material name="HubcapYellow">
-					<color rgba="1.0 0.811 0.151 1.0" />
-				</material>
-			</visual>
-			<collision>
-				<origin xyz="0 0 0" rpy="0 0 0" />
-				<geometry>
-					<box size="0.01 0.01 0.01" />
-				</geometry>
-			</collision>
-		</link>
-		<joint name="base_${suffix}_wheel_joint" type="continuous">
-			<axis xyz="0 1 0" />
-			<anchor xyz="0 0 0" />
-			<limit effort="100" velocity="100" />
-			<joint_properties damping="0.0" friction="0.0" />
-			<origin xyz="0 ${reflect*0.158} 0.091" rpy="0 0 0" />
-			<parent link="base_link" />
+			<parent link="p3dx_${suffix}_hubcap" />
 			<child link="p3dx_${suffix}_wheel" />
 		</joint>
 		<!-- gazebo elements -->
-    <transmission name="${parent}_${suffix}_wheel_trans">
-      <type>pr2_mechanism_model/SimpleTransmission</type>
-      <joint name="base_${suffix}_wheel_joint" />
-      <actuator name="base_${suffix}_wheel_motor">
-        <hardwareInterface>EffortJointInterface</hardwareInterface>
-        <mechanicalReduction>${reflect * 624/35 * 80/19}</mechanicalReduction>
-      </actuator>
-    </transmission>
+		<transmission name="${parent}_${suffix}_wheel_trans">
+			<type>pr2_mechanism_model/SimpleTransmission</type>
+			<joint name="base_${suffix}_wheel_joint" />
+			<actuator name="base_${suffix}_wheel_motor">
+				<hardwareInterface>EffortJointInterface</hardwareInterface>
+				<mechanicalReduction>${reflect * 624/35 * 80/19}</mechanicalReduction>
+			</actuator>
+		</transmission>
 		<gazebo reference="p3dx_${suffix}_hubcap">
 			<material>Gazebo/Yellow</material>

Commit message: Fixed wheel collision with ground

File: p3dx_description/urdf/p3dx_wheel.xacro (robot description, xacro)
@@ -56,5 +56,5 @@
 				<origin xyz="0 0 0" rpy="${-3.1415927/2} 0 0" />
 				<geometry>
-					<mesh filename="file://$(find p3dx_description)/meshes/${suffix}_wheel.stl"/>
+					<!-- <mesh filename="file://$(find p3dx_description)/meshes/${suffix}_wheel.stl"/> -->
 					<cylinder radius="0.09" length="0.01" />
 				</geometry>
