Commit message: Changed box 0 to avoid Assertion _size[0] > 0 failed

File: p3dx_description/urdf/p3dx.xacro (robot description, xacro)
@@ -76,5 +76,5 @@
 			<origin xyz="0 0 0" rpy="0 0 0" />
 			<geometry>
-				<box size="0 0 0" />
+				<box size="0.01 0.01 0.01" />
 			</geometry>
 		</collision>
@@ -109,5 +109,5 @@
 			<origin xyz="0 0 0" rpy="0 0 0" />
 			<geometry>
-				<box size="0 0 0" />
+				<box size="0.01 0.01 0.01" />
 			</geometry>
 		</collision>
@@ -172,5 +172,5 @@
 			<origin rpy="0 0 0" xyz="0 0 0" />
 			<geometry>
-				<box size="0 0 0" />
+				<box size="0.01 0.01 0.01" />
 			</geometry>
 		</collision>

File: p3dx_description/urdf/p3dx_wheel.xacro (robot description, xacro)
@@ -55,5 +55,5 @@
 				<origin xyz="0 0 0" rpy="0 0 0" />
 				<geometry>
-					<box size="0 0 0" />
+					<box size="0.01 0.01 0.01" />
 				</geometry>
 			</collision>

Commit message: Solved could not find mesh error

File: p3dx_description/urdf/p3dx.xacro (robot description, xacro)
@@ -16,5 +16,5 @@
 			<origin xyz="-0.045 0 0.148" rpy="0 0 0" />
 			<geometry name="pioneer_geom">
-				<mesh filename="package://p3dx_description/meshes/chassis.stl" />
+				<mesh filename="$(find p3dx_description)/meshes/chassis.stl" />
 			</geometry>
 			<material name="ChassisRed">
@@ -39,5 +39,5 @@
 			<origin xyz="0 0 0" rpy="0 0 0" />
 			<geometry name="top_geom">
-				<mesh filename="package://p3dx_description/meshes/top.stl" />
+				<mesh filename="$(find p3dx_description)/meshes/top.stl" />
 			</geometry>
 			<material name="TopBlack">
@@ -67,5 +67,5 @@
 			<origin xyz="0 0 0" rpy="0 0 0" />
 			<geometry name="pioneer_geom">
-				<mesh filename="package://p3dx_description/meshes/swivel.stl" />
+				<mesh filename="$(find p3dx_description)/meshes/swivel.stl" />
 			</geometry>
 			<material name="swivel">
@@ -100,5 +100,5 @@
 			<origin xyz="0 0 0" rpy="0 0 0" />
 			<geometry name="pioneer_geom">
-				<mesh filename="package://p3dx_description/meshes/center_hubcap.stl" />
+				<mesh filename="$(find p3dx_description)/meshes/center_hubcap.stl" />
 			</geometry>
 			<material name="swivel">
@@ -133,5 +133,5 @@
 			<origin xyz="0 0 0" rpy="0 0 0" />
 			<geometry name="pioneer_geom">
-				<mesh filename="package://p3dx_description/meshes/center_wheel.stl" />
+				<mesh filename="$(find p3dx_description)/meshes/center_wheel.stl" />
 			</geometry>
 			<material name="WheelBlack">
@@ -163,5 +163,5 @@
 			<origin rpy="0 0 0" xyz="0 0 0" />
 			<geometry name="pioneer_geom">
-				<mesh filename="package://p3dx_description/meshes/front_sonar.stl" />
+				<mesh filename="$(find p3dx_description)/meshes/front_sonar.stl" />
 			</geometry>
 			<material name="SonarYellow">
@@ -191,5 +191,5 @@
 			<origin xyz="0 0 0" rpy="0 0 0" />
 			<geometry>
-				<mesh filename="package://p3dx_description/meshes/lms100.dae" />
+				<mesh filename="$(find p3dx_description)/meshes/lms100.dae" />
 			</geometry>
 		</visual>

File: p3dx_description/urdf/p3dx_wheel.xacro (robot description, xacro)
@@ -16,5 +16,5 @@
 				<origin xyz="0 0 0" rpy="0 0 0" />
 				<geometry name="pioneer_geom">
-					<mesh filename="package://p3dx_description/meshes/${suffix}_wheel.stl" />
+					<mesh filename="$(find p3dx_description)/meshes/${suffix}_wheel.stl" />
 				</geometry>
 				<material name="WheelBlack">
@@ -25,5 +25,5 @@
 				<origin xyz="0 0 0" rpy="${-3.1415927/2} 0 0" />
 				<geometry>
-					<!--<mesh filename="package://p3dx_description/meshes/${suffix}_wheel.stl"/> -->
+					<!--<mesh filename="$(find p3dx_description)/meshes/${suffix}_wheel.stl"/> -->
 					<cylinder radius="0.09" length="0.01" />
 				</geometry>
@@ -46,5 +46,5 @@
 				<origin xyz="0 0 0" rpy="0 0 0" />
 				<geometry name="pioneer_geom">
-					<mesh filename="package://p3dx_description/meshes/${suffix}_hubcap.stl" />
+					<mesh filename="$(find p3dx_description)/meshes/${suffix}_hubcap.stl" />
 				</geometry>
 				<material name="HubcapYellow">

Commit message: Modified changes for correct rotation

File: p3dx_description/urdf/p3dx.xacro (robot description, xacro)
@@ -1,17 +1,17 @@
 <?xml version="1.0"?>
 <robot name="p3dx" xmlns:xacro="http://ros.org/wiki/xacro">
-  <!-- import all gazebo-customization elements, including gazebo colors -->
-  <xacro:include filename="$(find p3dx_description)/urdf/gz.xacro" />
-  <!-- import the pioneer 3dx's wheels -->
-  <xacro:include filename="$(find p3dx_description)/urdf/p3dx_wheel.xacro" />
-  <!-- chassis -->
+	<!-- import all gazebo-customization elements, including gazebo colors -->
+	<xacro:include filename="$(find p3dx_description)/urdf/gz.xacro" />
+	<!-- import the pioneer 3dx's wheels -->
+	<xacro:include filename="$(find p3dx_description)/urdf/p3dx_wheel.xacro" />
+	<!-- chassis -->
 	<link name="base_link">
 		<inertial>
 			<mass value="3.5" />
-			<!--<origin xyz="-0.025 0 -0.223"/> -->
+			<origin xyz="-0.025 0 -0.223"/>
 			<origin xyz="-0.05 0 0" />
 			<inertia ixx="1" ixy="0" ixz="0" iyy="1" iyz="0" izz="1" />
 		</inertial>
-		<visual name="base_visual">
+		<visual name="base_link">
 			<origin xyz="-0.045 0 0.148" rpy="0 0 0" />
 			<geometry name="pioneer_geom">
@@ -29,5 +29,5 @@
 		</collision>
 	</link>
-  <!-- top_plate -->
+	<!-- top_plate -->
 	<link name="top_plate">
 		<inertial>
@@ -57,5 +57,5 @@
 		<child link="top_plate" />
 	</joint>
-  <!-- swivel -->
+	<!-- swivel -->
 	<link name="swivel">
 		<inertial>
@@ -80,5 +80,5 @@
 		</collision>
 	</link>
-	<joint name="base_swivel_joint" type="continuous">
+	<joint name="base_swivel_joint" type="fixed">
 		<origin xyz="-0.185 0 0.055" rpy="0 0 0" />
 		<axis xyz="0 0 1" />
@@ -89,5 +89,5 @@
 		<child link="swivel" />
 	</joint>
-  <!-- center_hubcap -->
+	<!-- center_hubcap -->
 	<link name="center_hubcap">
 		<inertial>
@@ -122,5 +122,5 @@
 		<child link="center_wheel" />
 	</joint>
-  <!-- center_wheel -->
+	<!-- center_wheel -->
 	<link name="center_wheel">
 		<inertial>
@@ -147,11 +147,11 @@
 	</link>
 	<joint name="center_wheel_joint" type="fixed">
-		<origin xyz="-0.0035 0 -0.001" rpy="0 0 0"/>
-		<parent link="center_wheel"/>
-		<child link="center_hubcap"/>
-	</joint>
-	<xacro:p3dx_wheel suffix="left" parent="base_link" reflect="1"/>
-	<xacro:p3dx_wheel suffix="right" parent="base_link" reflect="-1"/>
-  <!-- front_sonar -->
+		<origin xyz="-0.0035 0 -0.001" rpy="0 0 0" />
+		<parent link="center_wheel" />
+		<child link="center_hubcap" />
+	</joint>
+	<xacro:p3dx_wheel suffix="left" parent="base_link" reflect="1" />
+	<xacro:p3dx_wheel suffix="right" parent="base_link" reflect="-1" />
+	<!-- front_sonar -->
 	<link name="front_sonar">
 		<inertial>

File: p3dx_description/urdf/p3dx_wheel.xacro (robot description, xacro)
@@ -28,5 +28,5 @@
 			</collision>
 		</link>
-		<joint name="base_${suffix}_hubcap_joint" type="continuous">
+		<joint name="base_${suffix}_hubcap_joint" type="fixed">
 			<axis xyz="0 1 0" />
 			<anchor xyz="0 0 0" />
@@ -61,8 +61,10 @@
 			</collision>
 		</link>
-		<joint name="base_${suffix}_wheel_joint" type="fixed">
+		<joint name="base_${suffix}_wheel_joint" type="continuous">
 			<origin xyz="0 0 0" rpy="0 0 0" />
 			<parent link="p3dx_${suffix}_hubcap" />
 			<child link="p3dx_${suffix}_wheel" />
+			<axis xyz="0 1 0" rpy="0 0 0"/>
+			<!-- <limit lower="-1.57" upper="1.57" effort="10.0" velocity="1.0"/> -->
 		</joint>
 		<!-- gazebo elements -->

Commit message: Removed dummy joint

File: p3dx_description/urdf/p3dx.xacro (robot description, xacro)
@@ -6,5 +6,4 @@
 	<xacro:include filename="$(find p3dx_description)/urdf/p3dx_wheel.xacro" />
 	<!-- chassis -->
-	<link name="base" />
 	<link name="base_link">
 		<inertial>
@@ -30,9 +29,4 @@
 		</collision>
 	</link>
-	<joint name="base_footprint_joint" type="fixed">
-		<origin xyz="0 0 0" rpy="0 0 0" />
-		<parent link="base" />
-		<child link="base_link" />
-	</joint>
 	<!-- top_plate -->
 	<link name="top_plate">
